Commit message: edit based on official UR description

File: ur_description_custom/urdf/ur5e_robotiq_85.urdf.xacro (robot description, xacro)
@@ -3,6 +3,8 @@
   <xacro:arg name="use_fake_hardware" default="true" />
   <xacro:arg name="sim_gazebo" default="false" />
+  <xacro:arg name="simulation_engine" default="mock" />
   <xacro:include filename="$(find ur_description)/urdf/ur_macro.xacro"/>
   <xacro:include filename="$(find robotiq_description)/urdf/robotiq_2f_85_macro.urdf.xacro"/>
+  <xacro:include filename="$(find ur_robotiq_moveit_config)/config/ur5_with_robotiq.ros2_control.xacro" />
   <link name="world" />
   <xacro:ur_robot
@@ -26,10 +28,14 @@
   </xacro:robotiq_gripper>
   <xacro:if value="$(arg use_fake_hardware)">
-    <xacro:include filename="$(find ur_robotiq_moveit_config)/config/ur5_with_robotiq.ros2_control.xacro" />
-    <xacro:ur5_with_robotiq_ros2_control name="FakeSystem" initial_positions_file="$(find ur_robotiq_moveit_config)/config/initial_positions.yaml"/>
+    <xacro:ur5_with_robotiq_ros2_control
+        name="FakeSystem"
+        initial_positions_file="$(find ur_robotiq_moveit_config)/config/initial_positions.yaml"
+        simulation_engine="$(arg simulation_engine)"/>
   </xacro:if>
   <xacro:if value="$(arg sim_gazebo)">
-    <xacro:include filename="$(find ur_robotiq_moveit_config)/config/ur5e_robotiq_gazebo.ros2_control.xacro" />
-    <xacro:ur5_with_robotiq_gazebo_ros2_control name="GazeboSystem" initial_positions_file="$(find ur_robotiq_moveit_config)/config/initial_positions.yaml"/>
+    <xacro:ur5_with_robotiq_ros2_control
+        name="GazeboSystem"
+        initial_positions_file="$(find ur_robotiq_moveit_config)/config/initial_positions.yaml"
+        simulation_engine="$(arg simulation_engine)"/>
   </xacro:if>
 </robot>

File: ur_robotiq_moveit_config/config/ur5_with_robotiq.ros2_control.xacro (robot description, xacro)
@@ -1,10 +1,14 @@
 <?xml version="1.0"?>
 <robot xmlns:xacro="http://www.ros.org/wiki/xacro">
-    <xacro:macro name="ur5_with_robotiq_ros2_control" params="name initial_positions_file">
+    <xacro:macro name="ur5_with_robotiq_ros2_control" params="name initial_positions_file simulation_engine">
         <xacro:property name="initial_positions" value="${xacro.load_yaml(initial_positions_file)['initial_positions']}"/>
         <ros2_control name="${name}" type="system">
             <hardware>
-                <!-- Use mock components for MoveIt demo -->
-                <plugin>mock_components/GenericSystem</plugin>
+                <xacro:if value="${simulation_engine == 'mock'}">
+                    <plugin>mock_components/GenericSystem</plugin>
+                </xacro:if>
+                <xacro:if value="${simulation_engine == 'gazebo'}">
+                    <plugin>gazebo_ros2_control/GazeboSystem</plugin>
+                </xacro:if>
             </hardware>
             <joint name="shoulder_pan_joint">
